File: mcu.kicad_sch (KiCad schematic)
At the start: 29 parts, among them U3 ESP32-C3, U4 W25Q128JVS, Y1 40Mhz

Commit message: Checking in before submitting rev.5 to JLCPCB.
Parts:
- added R11: 499R, Resistor_SMD:R_0201_0603Metric, symbol Device:R
- BOOT1, PU1: footprint TestPoint:TestPoint_Pad_1.5x1.5mm -> TestPoint:TestPoint_Pad_D1.0mm; now left out of the parts list
- Y1: footprint firefly:Crystal_SeikoEpson_FA20H -> Crystal:Crystal_SMD_2520-4Pin_2.5x2.0mm; MPN C255973 -> C409424; MPN_old (none) -> C255973
- renumbered C16 to C10, C10 to C11, C2 to C12, C4 to C14, C311 to C15, C312 to C16, C15 to C17, C9 to C5, C11 to C6, C6 to C7, C12 to C8, C14 to C9, R308 to R10, R2 to R3, R5 to R4, R303 to R5, R304 to R6, R305 to R7, R306 to R8, R307 to R9, U4 to U3, U3 to U4
Connections:
- net IO20: now reaches U4.27 (U0RXD/GPIO20)
- net at U4.28 (U0TXD/GPIO21): now also R11.1
- new net IO21: R11.2
- no-connect marks 4 -> 2
