File: mcu.kicad_sch (KiCad schematic)
At the start: 30 parts, among them U3 W25Q128JVS, U4 ESP32-C3, Y1 40Mhz

Commit message: Use ESP suggested C3 footprint and update for KiCad 8.
Parts:
- U4: footprint Package_DFN_QFN:QFN-32-1EP_5x5mm_P0.5mm_EP3.1x3.1mm -> Package_DFN_QFN:QFN-32-1EP_5x5mm_P0.5mm_EP3.45x3.45mm
- Y1: footprint Crystal:Crystal_SMD_2520-4Pin_2.5x2.0mm -> firefly:crystal_2520
Changed lines of the file:
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@@
 			)
 		)
-		(property "Footprint" "Crystal:Crystal_SMD_2520-4Pin_2.5x2.0mm"
+		(property "Footprint" "firefly:crystal_2520"
 			(at 48.26 166.37 0)
 			(effects
@@
 			)
 		)
-		(property "Footprint" "Package_DFN_QFN:QFN-32-1EP_5x5mm_P0.5mm_EP3.1x3.1mm"
+		(property "Footprint" "Package_DFN_QFN:QFN-32-1EP_5x5mm_P0.5mm_EP3.45x3.45mm"
 			(at 149.86 121.92 0)
 			(effects
