File: output.kicad_sch (KiCad schematic)
At the start: 5 parts, among them U401 SN74LVC1T45DBV

Commit message: Checking in before submitting rev.5 to JLCPCB.
Parts:
- added C19, C20: 100n, Capacitor_SMD:C_0201_0603Metric, symbol Device:C
- added D2, D3, D4: WS2812B, firefly:WS2812B, symbol Firefly:WS2812B
- renumbered C8 to C18, J401 to J2, R4 to R12, U401 to U5
Connections:
- net 3V3: now also C19.1
- net 5V: now also C20.1, D2.4 (VDD), D3.4 (VDD), D4.4 (VDD)
- net GND: now also C19.2, C20.2, D2.2 (GND), D3.2 (GND), D4.2 (GND)
- net at D1.1 (D0): now also D2.3 (DIN)
- new net: D3.1 (D0), D4.3 (DIN)
- new net: D2.1 (D0), D3.3 (DIN)
Other:
- moved on the sheet: D1, U5

Commit message: JLCPCB submit
Parts:
- J2: footprint firefly:THD_FPC_24 -> firefly:JUSHUO_FPC_24; MPN C283150 -> C262669
Changed lines of the file:
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@@
       (effects (font (size 1.27 1.27)))
     )
-    (property "Footprint" "firefly:THD_FPC_24" (at 76.2 66.04 0)
+    (property "Footprint" "firefly:JUSHUO_FPC_24" (at 76.2 66.04 0)
       (effects (font (size 1.27 1.27)) hide)
     )
@@
       (effects (font (size 1.27 1.27)) hide)
     )
-    (property "MPN" "C283150" (at 78.74 67.31 0)
+    (property "MPN" "C262669" (at 78.74 67.31 0)
       (effects (font (size 1.27 1.27)) hide)
     )
