File: power.kicad_sch (KiCad schematic)
At the start: 10 parts, among them U1 SPX3819M5-L-3-3, U2 USBLC6-2SC6

Commit message: Checking in before submitting rev.5 to JLCPCB.
Parts:
- added 3V1, 5V1: TestPoint, TestPoint:TestPoint_Pad_1.0x1.0mm, symbol Connector:TestPoint
- GND1: footprint TestPoint:TestPoint_Pad_1.5x1.5mm -> TestPoint:TestPoint_Pad_1.0x1.0mm; now left out of the parts list
- renumbered C3 to C2, C5 to C3, C7 to C4, R3 to R2, U2 to U1, U1 to U2
Connections:
- net 3V3: now also 3V1.1
- net 5V: now also 5V1.1
Other:
- moved on the sheet: GND1
